Commit message: 接口修复

File: SimEnv/src/unitree_guide/unitree_ros/robots/a1_description/xacro/robot.xacro (robot description, xacro)
@@ -1,11 +1,13 @@
 <?xml version="1.0"?>
 <robot name="a1" xmlns:xacro="http://www.ros.org/wiki/xacro">
-    <!--
-      A1 机器人结构定义。
-      multi_floor_gazeboSim.launch 会用 xacro 展开本文件生成 robot_description，
-      再由 gazebo_ros/spawn_model 插入 Gazebo。Gazebo 插件和传感器话题在
-      gazebo.xacro 中定义，这里主要定义 link/joint 和传感器安装位置。
-    -->
     <xacro:arg name="DEBUG" default="false"/>
+    <xacro:arg name="ENABLE_SENSOR_DATA" default="true"/>
+    <xacro:arg name="ENABLE_LIVOX" default="$(arg ENABLE_SENSOR_DATA)"/>
+    <xacro:arg name="ENABLE_LIVOX_IMU" default="$(arg ENABLE_LIVOX)"/>
+    <xacro:arg name="ENABLE_REALSENSE" default="$(arg ENABLE_SENSOR_DATA)"/>
+    <xacro:arg name="ENABLE_FRONT_CAMERA" default="false"/>
+    <xacro:arg name="ENABLE_GROUND_TRUTH" default="true"/>
+    <xacro:arg name="ENABLE_FOOT_CONTACT_SENSOR" default="false"/>
+    <xacro:arg name="ENABLE_FOOT_FORCE_VISUAL" default="false"/>
     <xacro:include filename="$(find a1_description)/xacro/const.xacro"/>
     <xacro:include filename="$(find a1_description)/xacro/materials.xacro"/>
@@ -18,5 +20,5 @@
     <xacro:property name="rolloverProtection" value="false"/>
     <!-- Debug mode will hung up the robot, use "true" or "false" to switch it. -->
-    <xacro:if value="$(arg DEBUG)">
+    <xacro:if value="${'$(arg DEBUG)' == 'true'}">
         <link name="world"/>
         <joint name="base_static_joint" type="fixed">
@@ -116,116 +118,150 @@
         </collision>
     </link>
-    <!--
-      Livox Mid-360 的实体 link。
-      gazebo.xacro 会在 reference="laser_livox" 上挂 ray 传感器插件，
-      最终向 /scan 发布原始点云。
-    -->
+    <!-- livox mid360 -->
     <link name="laser_livox">
             <collision>
-            <origin xyz="0 0 0" rpy="0 0 0"/>
-            <geometry>
+                <origin xyz="0 0 0" rpy="0 0 0"/>
+                <geometry>
                     <mesh filename="package://a1_description/meshes/livox_mid360.dae"/>
-            </geometry>
-            </collision>
-            <visual>
-            <origin xyz="0.0 0 0" rpy="0 0 0"/>
-            <geometry>
+                </geometry>
+            </collision>
+            <visual>
+                <origin xyz="0.0 0 0" rpy="0 0 0"/>
+                <geometry>
                     <mesh filename="package://a1_description/meshes/livox_mid360.dae"/>
-            </geometry>
-            </visual>
-    </link>
-    <!-- Livox 与 base 固连；这里的 rpy 体现雷达安装俯仰角。 -->
-    <joint name="laser_livox_joint" type="fixed" >
-        <origin xyz="0.2 0 0.08" rpy="0 0.785 0" />
-        <parent link="base" />
-        <child link="laser_livox"/>
-    </joint>
-    <!-- Livox 内置 IMU 的简化 link，对应 gazebo.xacro 里的 /livox/imu 插件。 -->
+                </geometry>
+            </visual>
+    </link>
+    <joint name="laser_livox_joint" type="fixed">
+            <origin xyz="0.2 0 0.08" rpy="0 0.785 0"/>
+            <parent link="base"/>
+            <child link="laser_livox"/>
+    </joint>
+    <!-- livox mid360-imu -->
     <link name="livox_imu_link">
-        <inertial>
-            <mass value="0.001"/>
-            <origin rpy="0 0 0" xyz="0 0 0"/>
-            <inertia ixx="0.0001" ixy="0" ixz="0" iyy="0.0001" iyz="0" izz="0.0001"/>
-        </inertial>
-        <visual>
-            <origin rpy="0 0 0" xyz="0 0 0"/>
-            <geometry>
-                <box size="0.001 0.001 0.001"/>
-            </geometry>
-            <!-- <material name="red"/> -->
-        </visual>
-        <collision>
-            <origin rpy="0 0 0" xyz="0 0 0"/>
-            <geometry>
-                <box size=".001 .001 .001"/>
-            </geometry>
-        </collision>
-    </link>
-     <!-- IMU 相对 Livox 外壳的安装偏移。 -->
-     <joint name="livox_imu_joint" type="fixed">
-        <parent link="laser_livox"/>
-        <child link="livox_imu_link"/>
-        <origin rpy="0 0 0" xyz="-0.011 -0.02329 0.04412"/>
-    </joint>
-    <!--
-      RealSense D415 深度相机 link。
-      gazebo.xacro 会在 reference="real_sense" 上挂 openni/kinect 插件，
-      发布 /real_sense/rgb/image_raw、/real_sense/depth/image_raw、
-      /real_sense/depth/points 等话题。
-    -->
-    <link
-        name="real_sense">
-        <inertial>
-        <origin
-            xyz="-0.00975078931607951 0.00306064913353049 -7.04374991291334E-05"
-            rpy="0 0 0" />
-        <mass
-            value="0.103311749598955" />
-        <inertia
-            ixx="7.35323632954531E-05"
-            ixy="3.0437488683846E-06"
-            ixz="2.08538534427428E-08"
-            iyy="7.40427481540393E-06"
-            iyz="-1.93018760531168E-08"
-            izz="7.2832884533889E-05" />
-        </inertial>
-        <visual>
-        <origin
-            xyz="0 0 0"
-            rpy="0 0 1.5708" />
-        <geometry>
-            <mesh
-            filename="package://a1_description/meshes/d415.stl" />
-        </geometry>
-        <material
-            name="">
-            <color
-            rgba="0.666666666666667 0.698039215686274 0.768627450980392 1" />
-        </material>
-        </visual>
-        <collision>
-        <origin
-            xyz="0 0 0"
-            rpy="0 0 0" />
-        <geometry>
-            <mesh
-            filename="package://a1_description/meshes/d415.stl" />
-        </geometry>
-        </collision>
-    </link>
-    <joint
-        name="real_sense_joint"
-        type="fixed">
-        <!-- 相机安装在机身前方，算法看到的深度/图像视角由此决定。 -->
-        <origin
-        xyz="0.28 0 0.043"
-        rpy="0 0 0" />
-        <parent
-        link="base" />
-        <child
-        link="real_sense" />
-        <axis
-        xyz="0 0 1" />
-    </joint>
+            <inertial>
+                <mass value="0.001"/>
+                <origin rpy="0 0 0" xyz="0 0 0"/>
+                <inertia ixx="0.0001" ixy="0" ixz="0" iyy="0.0001" iyz="0" izz="0.0001"/>
+            </inertial>
+            <visual>
+                <origin rpy="0 0 0" xyz="0 0 0"/>
+                <geometry>
+                    <box size="0.001 0.001 0.001"/>
+                </geometry>
+            </visual>
+            <collision>
+                <origin rpy="0 0 0" xyz="0 0 0"/>
+                <geometry>
+                    <box size=".001 .001 .001"/>
+                </geometry>
+            </collision>
+    </link>
+    <joint name="livox_imu_joint" type="fixed">
+            <parent link="laser_livox"/>
+            <child link="livox_imu_link"/>
+            <origin rpy="0 0 0" xyz="-0.011 -0.02329 0.04412"/>
+    </joint>
+    <!-- depth camera -->
+    <link name="real_sense">
+            <inertial>
+                <origin xyz="-0.00975078931607951 0.00306064913353049 -7.04374991291334E-05" rpy="0 0 0"/>
+                <mass value="0.103311749598955"/>
+                <inertia
+                    ixx="7.35323632954531E-05"
+                    ixy="3.0437488683846E-06"
+                    ixz="2.08538534427428E-08"
+                    iyy="7.40427481540393E-06"
+                    iyz="-1.93018760531168E-08"
+                    izz="7.2832884533889E-05"/>
+            </inertial>
+            <visual>
+                <origin xyz="0 0 0" rpy="0 0 1.5708"/>
+                <geometry>
+                    <mesh filename="package://a1_description/meshes/d415.stl"/>
+                </geometry>
+                <material name="">
+                    <color rgba="0.666666666666667 0.698039215686274 0.768627450980392 1"/>
+                </material>
+            </visual>
+            <collision>
+                <origin xyz="0 0 0" rpy="0 0 0"/>
+                <geometry>
+                    <mesh filename="package://a1_description/meshes/d415.stl"/>
+                </geometry>
+            </collision>
+    </link>
+    <joint name="real_sense_joint" type="fixed">
+            <origin xyz="0.28 0 0.043" rpy="0 0 0"/>
+            <parent link="base"/>
+            <child link="real_sense"/>
+            <axis xyz="0 0 1"/>
+    </joint>
+    <link name="real_sense_optical_frame"/>
+    <joint name="real_sense_optical_joint" type="fixed">
+            <parent link="real_sense"/>
+            <child link="real_sense_optical_frame"/>
+            <!-- ROS optical frame: X right, Y down, Z forward. -->
+            <origin xyz="0 0 0" rpy="-1.57079632679 0 -1.57079632679"/>
+    </joint>
+    <xacro:if value="${'$(arg ENABLE_FRONT_CAMERA)' == 'true'}">
+        <!-- optional front monocular camera -->
+        <link name="front_camera">
+            <inertial>
+                <mass value="0.001"/>
+                <origin rpy="0 0 0" xyz="0 0 0"/>
+                <inertia ixx="0.0001" ixy="0" ixz="0" iyy="0.0001" iyz="0" izz="0.0001"/>
+            </inertial>
+            <visual>
+                <origin rpy="0 0 0" xyz="0 0 0"/>
+                <geometry>
+                    <box size="0.02 0.02 0.02"/>
+                </geometry>
+                <material name="black"/>
+            </visual>
+        </link>
+        <joint name="front_camera_joint" type="fixed">
+            <origin xyz="0.30 0 0.08" rpy="0 0 0"/>
+            <parent link="base"/>
+            <child link="front_camera"/>
+        </joint>
+        <gazebo reference="front_camera">
+            <material>Gazebo/Grey</material>
+            <sensor type="camera" name="camera">
+                <update_rate>30.0</update_rate>
+                <camera name="head">
+                    <horizontal_fov>1.3962634</horizontal_fov>
+                    <image>
+                        <width>800</width>
+                        <height>800</height>
+                        <format>R8G8B8</format>
+                    </image>
+                    <clip>
+                        <near>0.02</near>
+                        <far>300</far>
+                    </clip>
+                    <noise>
+                        <type>gaussian</type>
+                        <mean>0.0</mean>
+                        <stddev>0.007</stddev>
+                    </noise>
+                </camera>
+                <plugin name="camera_controller" filename="libgazebo_ros_camera.so">
+                    <alwaysOn>true</alwaysOn>
+                    <updateRate>0.0</updateRate>
+                    <cameraName>camera</cameraName>
+                    <imageTopicName>image_raw</imageTopicName>
+                    <cameraInfoTopicName>camera_info</cameraInfoTopicName>
+                    <frameName>front_camera</frameName>
+                    <hackBaseline>0.07</hackBaseline>
+                    <distortionK1>0.0</distortionK1>
+                    <distortionK2>0.0</distortionK2>
+                    <distortionK3>0.0</distortionK3>
+                    <distortionT1>0.0</distortionT1>
+                    <distortionT2>0.0</distortionT2>
+                </plugin>
+            </sensor>
+        </gazebo>
+    </xacro:if>
     <xacro:leg name="FR" mirror="-1" mirror_dae="False" front_hind="1" front_hind_dae="True">
         <origin rpy="0 0 0" xyz="${leg_offset_x} ${-leg_offset_y} 0"/>
